File: sunlight_pcb.kicad_pcb (KiCad board)
At the start: 2 copper layers, 136.5 x 127 mm, 17 parts, among them J1 Conn_01x01, J2 Conn_01x01, J3 Conn_01x01, J4 Conn_01x01, J6 PJ-036AH-SMT-TR, Q1 DMN63D8LW, Q2 DMN63D8LW, U1 LDH-65-700, U2 LDH-65-700, U3 SeeedStudio ESP32-C3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

Commit message: change barrel to tht and update 3d models
Parts:
- removed J6: PJ-036AH-SMT-TR, Connector_BarrelJack:BarrelJack_CUI_PJ-036AH-SMT_Horizontal
- added J8: PJ-002AH, sunlight_pcb:CUI_PJ-002AH, F.Cu at (64.2, 81.0)
Changed lines of the file:
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@@
   (net 28 "Net-(D1-K)")
   (net 29 "unconnected-(U3-GND-Pad20)")
+  (net 30 "unconnected-(J8-Pad3)")
   (footprint "Capacitor_SMD:CP_Elec_5x5.3" (layer "F.Cu")
     (at 89.7 96.5)
@@
     )
   )
-  (footprint "Connector_BarrelJack:BarrelJack_CUI_PJ-036AH-SMT_Horizontal" (layer "F.Cu")
-    (at 69.55 72.3)
-    (descr "Surface-mount DC Barrel Jack, http://www.cui.com/product/resource/pj-036ah-smt.pdf")
-    (tags "Power Jack SMT")
+  (footprint "sunlight_pcb:CUI_PJ-002AH" (layer "F.Cu")
+    (at 64.2 80.95)
     (property "Sheetfile" "sunlight_pcb.kicad_sch")
     (property "Sheetname" "")
-    (property "ki_description" "DC Barrel Jack")
-    (property "ki_keywords" "DC power barrel jack connector")
-    (attr smd)
-    (fp_text reference "J6" (at -4.5 -5.75) (layer "F.SilkS")
-        (effects (font (size 1 1) (thickness 0.15)))
-    )
-    (fp_text value "PJ-036AH-SMT-TR\n" (at 0 11.25) (layer "F.Fab")
-        (effects (font (size 1 1) (thickness 0.15)))
-    )
-    (fp_text user "${REFERENCE}" (at 0 0) (layer "F.Fab")
-        (effects (font (size 1 1) (thickness 0.15)))
-    )
-    (fp_line (start -4.6 -2.6) (end -4.2 -2.6)
-      (stroke (width 0.12) (type solid)) (layer "F.SilkS"))
-    (fp_line (start -4.6 -0.15) (end -4.6 -2.6)
-      (stroke (width 0.12) (type solid)) (layer "F.SilkS"))
-    (fp_line (start -4.6 10.1) (end -4.6 6.55)
-      (stroke (width 0.12) (type solid)) (layer "F.SilkS"))
-    (fp_line (start -4.2 -4.6) (end -1.2 -4.6)
-      (stroke (width 0.12) (type solid)) (layer "F.SilkS"))
-    (fp_line (start -4.2 -2.6) (end -4.2 -4.6)
-      (stroke (width 0.12) (type solid)) (layer "F.SilkS"))
-    (fp_line (start -1.19 -8.24) (end 0.55 -8.24)
-      (stroke (width 0.12) (type solid)) (layer "F.SilkS"))
-    (fp_line (start -1.19 -6.5) (end -1.19 -8.24)
-      (stroke (width 0.12) (type solid)) (layer "F.SilkS"))
-    (fp_line (start 2.6 -4.6) (end 4.2 -4.6)
-      (stroke (width 0.12) (type solid)) (layer "F.SilkS"))
-    (fp_line (start 4.2 -4.6) (end 4.2 -2.6)
-      (stroke (width 0.12) (type solid)) (layer "F.SilkS"))
-    (fp_line (start 4.2 -2.6) (end 4.6 -2.6)
-      (stroke (width 0.12) (type solid)) (layer "F.SilkS"))
-    (fp_line (start 4.6 -2.6) (end 4.6 -0.15)
-      (stroke (width 0.12) (type solid)) (layer "F.SilkS"))
-    (fp_line (start 4.6 6.55) (end 4.6 10.1)
-      (stroke (width 0.12) (type solid)) (layer "F.SilkS"))
-    (fp_line (start 4.6 10.1) (end -4.6 10.1)
-      (stroke (width 0.12) (type solid)) (layer "F.SilkS"))
-    (fp_line (start -8.9 -8.5) (end -8.9 10.5)
-      (stroke (width 0.05) (type solid)) (layer "F.CrtYd"))
-    (fp_line (start -8.9 10.5) (end 8.9 10.5)
-      (stroke (width 0.05) (type solid)) (layer "F.CrtYd"))
-    (fp_line (start 8.9 -8.5) (end -8.9 -8.5)
-      (stroke (width 0.05) (type solid)) (layer "F.CrtYd"))
-    (fp_line (start 8.9 10.5) (end 8.9 -8.5)
-      (stroke (width 0.05) (type solid)) (layer "F.CrtYd"))
-    (fp_line (start -4.5 -2.5) (end -4.5 10)
-      (stroke (width 0.1) (type solid)) (layer "F.Fab"))
-    (fp_line (start -4.5 10) (end 4.5 10)
-      (stroke (width 0.1) (type solid)) (layer "F.Fab"))
-    (fp_line (start -4.1 -4.5) (end -4.1 -2.5)
-      (stroke (width 0.1) (type solid)) (layer "F.Fab"))
-    (fp_line (start -4.1 -2.5) (end -4.5 -2.5)
-      (stroke (width 0.1) (type solid)) (layer "F.Fab"))
-    (fp_line (start 4.1 -4.5) (end -4.1 -4.5)
-      (stroke (width 0.1) (type solid)) (layer "F.Fab"))
-    (fp_line (start 4.1 -2.5) (end 4.1 -4.5)
-      (stroke (width 0.1) (type solid)) (layer "F.Fab"))
-    (fp_line (start 4.5 -2.5) (end 4.1 -2.5)
-      (stroke (width 0.1) (type solid)) (layer "F.Fab"))
-    (fp_line (start 4.5 10) (end 4.5 -2.5)
-      (stroke (width 0.1) (type solid)) (layer "F.Fab"))
-    (fp_circle (center 0.7 -3.4) (end 0.75 -2.95)
-      (stroke (width 0.12) (type solid)) (fill none) (layer "F.Fab"))
-    (pad "" np_thru_hole circle (at 0 7) (size 2 2) (drill 2) (layers "*.Cu" "*.Mask"))
-    (pad "1" smd rect (at 0.7 -5.8) (size 3.3 4.4) (layers "F.Cu" "F.Paste" "F.Mask")
-      (net 4 "+24V") (pintype "passive"))
-    (pad "2" smd rect (at -6.45 3.2) (size 3.9 6.2) (layers "F.Cu" "F.Paste" "F.Mask")
-      (net 2 "GND") (pintype "passive"))
-    (pad "3" smd rect (at 6.45 3.2) (size 3.9 6.2) (layers "F.Cu" "F.Paste" "F.Mask"))
-    (model "${KIPRJMOD}/sunlight_pcb.pretty/CUI_DEVICES_PJ-036AH-SMT-TR.step"
-      (offset (xyz 0 -10 0))
+    (property "ki_keywords" "PJ-002AH")
+    (attr through_hole)
+    (fp_text reference "J8" (at 2.485118 -6.76532) (layer "F.SilkS")
+        (effects (font (size 1.000047 1.000047) (thickness 0.15)))
+    )
+    (fp_text value "PJ-002AH" (at 6.939165 5.78266) (layer "F.Fab")
+        (effects (font (size 1.001323 1.001323) (thickness 0.15)))
+    )
+    (fp_line (start -0.7 -4.5) (end 0.45 -4.5)
+      (stroke (width 0.127) (type solid)) (layer "F.SilkS"))
+    (fp_line (start -0.7 -2.55) (end -0.7 -4.5)
+      (stroke (width 0.127) (type solid)) (layer "F.SilkS"))
+    (fp_line (start -0.7 4.5) (end -0.7 2.65)
+      (stroke (width 0.127) (type solid)) (layer "F.SilkS"))
+    (fp_line (start 5.55 -4.5) (end 13.7 -4.5)
+      (stroke (width 0.127) (type solid)) (layer "F.SilkS"))
+    (fp_line (start 13.7 -4.5) (end 13.7 4.5)
+      (stroke (width 0.127) (type solid)) (layer "F.SilkS"))
+    (fp_line (start 13.7 4.5) (end -0.7 4.5)
+      (stroke (width 0.127) (type solid)) (layer "F.SilkS"))
+    (fp_circle (center -2 0) (end -1.8 0)
+      (stroke (width 0.4) (type solid)) (fill none) (layer "F.SilkS"))
+    (fp_line (start -1.55 -2.25) (end -1.55 2.35)
+      (stroke (width 0.05) (type solid)) (layer "F.CrtYd"))
+    (fp_line (start -1.55 2.35) (end -1 2.35)
+      (stroke (width 0.05) (type solid)) (layer "F.CrtYd"))
+    (fp_line (start -1 -4.75) (end 0.45 -4.75)
+      (stroke (width 0.05) (type solid)) (layer "F.CrtYd"))
+    (fp_line (start -1 -2.25) (end -1.55 -2.25)
+      (stroke (width 0.05) (type solid)) (layer "F.CrtYd"))
+    (fp_line (start -1 -2.25) (end -1 -4.75)
+      (stroke (width 0.05) (type solid)) (layer "F.CrtYd"))
+    (fp_line (start -1 4.75) (end -1 2.35)
+      (stroke (width 0.05) (type solid)) (layer "F.CrtYd"))
+    (fp_line (start 0.45 -6.1) (end 5.55 -6.1)
+      (stroke (width 0.05) (type solid)) (layer "F.CrtYd"))
+    (fp_line (start 0.45 -4.75) (end 0.45 -6.1)
+      (stroke (width 0.05) (type solid)) (layer "F.CrtYd"))
+    (fp_line (start 5.55 -6.1) (end 5.55 -4.75)
+      (stroke (width 0.05) (type solid)) (layer "F.CrtYd"))
+    (fp_line (start 5.55 -4.75) (end 14 -4.75)
+      (stroke (width 0.05) (type solid)) (layer "F.CrtYd"))
+    (fp_line (start 14 -4.75) (end 14 4.75)
+      (stroke (width 0.05) (type solid)) (layer "F.CrtYd"))
+    (fp_line (start 14 4.75) (end -1 4.75)
+      (stroke (width 0.05) (type solid)) (layer "F.CrtYd"))
+    (fp_line (start -0.7 -4.5) (end 13.7 -4.5)
+      (stroke (width 0.127) (type solid)) (layer "F.Fab"))
+    (fp_line (start -0.7 4.5) (end -0.7 -4.5)
+      (stroke (width 0.127) (type solid)) (layer "F.Fab"))
+    (fp_line (start 13.7 -4.5) (end 13.7 4.5)
+      (stroke (width 0.127) (type solid)) (layer "F.Fab"))
+    (fp_line (start 13.7 4.5) (end -0.7 4.5)
+      (stroke (width 0.127) (type solid)) (layer "F.Fab"))
+    (pad "1" thru_hole oval (at 0 0) (size 2.5 5) (drill oval 1 3.5) (layers "*.Cu" "*.Mask")
+      (net 4 "+24V") (pinfunction "1") (pintype "unspecified") (solder_mask_margin 0.102))
+    (pad "2" thru_hole oval (at 6 0) (size 2.25 4.5) (drill oval 1 3) (layers "*.Cu" "*.Mask")
+      (net 2 "GND") (pinfunction "2") (pintype "unspecified") (solder_mask_margin 0.102))
+    (pad "3" thru_hole oval (at 3 -4.7) (size 4.5 2.25) (drill oval 3 1) (layers "*.Cu" "*.Mask")
+      (net 30 "unconnected-(J8-Pad3)") (pinfunction "3") (pintype "unspecified+no_connect") (solder_mask_margin 0.102))
+    (model "${KIPRJMOD}/sunlight_pcb.pretty/CUI_DEVICES_PJ-002AH.step"
+      (offset (xyz 13.75 0 6.5))
       (scale (xyz 1 1 1))
       (rotate (xyz -90 0 0))
@@
     (pad "22" smd rect (at -4.5 -0.4 180) (size 2.3 1.3) (layers "F.Cu" "F.Paste" "F.Mask"))
     (pad "23" smd rect (at 2.1 0.6 180) (size 3.5 3.5) (layers "F.Cu" "F.Paste" "F.Mask"))
+    (model "${KIPRJMOD}/sunlight_pcb.pretty/Seeed Studio XIAO-ESP32-C3.step"
+      (offset (xyz 6.1 -1.7 0))
+      (scale (xyz 1 1 1))
+      (rotate (xyz -90 0 -90))
+    )
   )
   (gr_rect (start 53.5 24.5) (end 190 151.5)

Commit message: layout done, gerbers gened
Parts:
- added D1: D_Schottky, Diode_SMD:D_0603_1608Metric_Pad1.05x0.95mm_HandSolder, F.Cu at (85.5, 72.0)
- added J5: NTC, sunlight_pcb:SolderNTC-1.27mm, F.Cu at (84.5, 113.5)
- added J7: Conn_01x02, Connector_PinHeader_2.54mm:PinHeader_1x02_P2.54mm_Vertical, F.Cu at (84.5, 107.7)
- added R2: 10k, Diode_SMD:D_0603_1608Metric_Pad1.05x0.95mm_HandSolder, F.Cu at (106.0, 86.0)
- added R3: 10k, Diode_SMD:D_0603_1608Metric_Pad1.05x0.95mm_HandSolder, F.Cu at (106.0, 82.0)
- added REF**: MountingHole_3.2mm_M3, MountingHole:MountingHole_3.2mm_M3, F.Cu at (186.5, 135.0)
- added REF**: MountingHole_3.2mm_M3, MountingHole:MountingHole_3.2mm_M3, F.Cu at (186.5, 45.0)
- added REF**: MountingHole_3.2mm_M3, MountingHole:MountingHole_3.2mm_M3, F.Cu at (86.5, 135.0)
- added REF**: MountingHole_3.2mm_M3, MountingHole:MountingHole_3.2mm_M3, F.Cu at (86.5, 45.0)
- added TP1: TestPoint, TestPoint:TestPoint_Pad_1.0x1.0mm, F.Cu at (84.5, 66.5)
- added TP2: TestPoint, TestPoint:TestPoint_Pad_1.0x1.0mm, F.Cu at (90.5, 114.0)
- added TP3: TestPoint, TestPoint:TestPoint_Pad_1.0x1.0mm, F.Cu at (84.5, 57.0)
- added TP4: TestPoint, TestPoint:TestPoint_Pad_1.0x1.0mm, F.Cu at (84.5, 61.8)
- C1: footprint Capacitor_SMD:C_0402_1005Metric -> Capacitor_SMD:C_0603_1608Metric_Pad1.08x0.95mm_HandSolder
- J1, J2, J3, J4: footprint Connector_Wire:SolderWire-0.5sqmm_1x01_D0.9mm_OD2.1mm -> Connector_Wire:SolderWire-2sqmm_1x01_D2mm_OD3.9mm
- R1: footprint Resistor_SMD:R_0402_1005Metric -> Resistor_SMD:R_0603_1608Metric_Pad0.98x0.95mm_HandSolder
- moved J2 107.8 mm to (186.5, 83.0), turned to 180 degrees
- moved J1 106.8 mm to (186.5, 73.0), turned to 180 degrees
- moved J4 90.3 mm to (186.5, 107.0)
- moved J3 90.0 mm to (186.5, 97.0)
- moved C5 52.9 mm to (102.5, 52.0), turned to -90 degrees
- moved U3 42.2 mm to (94.2, 83.5), turned to 90 degrees
- moved R1 37.4 mm to (90.0, 108.5), turned to 180 degrees
- moved J8 36.8 mm to (96.3, 98.8), turned to 180 degrees
- moved C1 35.1 mm to (90.0, 106.5)
- moved C2 34.0 mm to (90.5, 62.5), turned to -90 degrees
- moved C3 21.7 mm to (102.5, 100.0), turned to -90 degrees
- moved U4 21.4 mm to (100.0, 62.5)
- moved Q1 17.3 mm to (95.5, 111.0), turned to -90 degrees
- moved Q2 17.0 mm to (104.0, 71.0)
- moved C6 12.9 mm to (102.5, 108.5), turned to -90 degrees
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Connections:
- J8 pad 3: unconnected-(J8-Pad3) -> GND
- U3 pad 1: Net-(J5-Pin_2) -> unconnected-(U3-PA02_A0_D0-Pad1)
- U3 pad 12: unconnected-(U3-3V3-Pad12) -> +3V3
- U3 pad 2: unconnected-(U3-PA4_A1_D1-Pad2) -> /UART_RX
- U3 pad 3: unconnected-(U3-PA10_A2_D2-Pad3) -> /UART_TX
- U3 pad 4: unconnected-(U3-PA11_A3_D3-Pad4) -> Net-(J5-Pin_2)
- U3 pad 6: /BLUE_INPUT -> unconnected-(U3-PA9_A5_D5_SCL-Pad6)
- U3 pad 7: /UART_TX -> unconnected-(U3-PB08_A6_D6_TX-Pad7)
- U3 pad 8: /UART_RX -> /BLUE_INPUT
Routing:
- net +3V3: track 0.00 -> 65.4 mm
- net /ORANGE_INPUT: track 0.00 -> 38.4 mm
- net /BLUE_INPUT: track 0.00 -> 33.6 mm
- net Net-(Q1-D): track 0.00 -> 31.2 mm
- net +5V: track 0.00 -> 31.0 mm
- net Net-(J5-Pin_2): track 0.00 -> 27.1 mm
- net /UART_TX: track 0.00 -> 21.0 mm
- net Net-(Q2-D): track 0.00 -> 20.5 mm, vias 0 -> 2
- net /UART_RX: track 0.00 -> 17.4 mm
- net GND: track 0.00 -> 10.4 mm, vias 0 -> 28
- net Net-(D1-K): track 0.00 -> 3.09 mm
- net Net-(J4-Pin_1): vias 0 -> 2
- net Net-(J3-Pin_1): vias 0 -> 2
- net Net-(J2-Pin_1): vias 0 -> 2
- net Net-(J1-Pin_1): vias 0 -> 2
- added copper zone on F.Cu, net +24V
- added copper zone on B.Cu, net GND
- added copper zone on F.Cu, net GND
- added copper zone on B.Cu, net Net-(J1-Pin_1)
- added copper zone on F.Cu, net Net-(J1-Pin_1)
- added copper zone on B.Cu, net Net-(J2-Pin_1)
- added copper zone on F.Cu, net Net-(J2-Pin_1)
- added copper zone on B.Cu, net Net-(J3-Pin_1)
- added copper zone on F.Cu, net Net-(J3-Pin_1)
- added copper zone on B.Cu, net Net-(J4-Pin_1)
- added copper zone on F.Cu, net Net-(J4-Pin_1)
Other:
- board size 136.5 x 127 mm -> 108 x 108 mm
- board text added: "5V"
- board text added: "BLUE"
- board text added: "GND"
- board text added: "GPIO"
- board text added: "NTC 10k"
- board text added: "ORANGE"
